File: Sensor-Board-KiCad7.0/Sensor board p2.kicad_sch (KiCad schematic)
At the start: 55 parts, among them U11 OPA396DCKT, U12 OPA396DCKT, U15 MMBFJ177LT1, U16 MMBFJ177LT1, U17 MMBFJ177LT1, U18 NAU7802SGI, U24 OPA396DCKT, U5 NAU7802SGI, U6 BME680, U7 OPA396DCKT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

Commit message: Added some part #
Added part numbers for resistors, capacitors, MOSFETS
Parts:
- C10, C11, C12, C13, C14, C5, C6, C7: LCSC (none) -> C14663
- R10, R11, R12, R13, R14, R15: LCSC (none) -> C22859
- R16, R17: LCSC (none) -> C23162
- R49, R50, R51: LCSC (none) -> C407640
- U15, U16, U17: LCSC (none) -> C106763
- U18, U5: Digikey (none) -> NAU7802SGITR-ND
- U6: LCSC (none) -> C125972
Changed lines of the file:
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@@
+      (effects (font (size 1.27 1.27)) hide)
+    )
+    (property "LCSC" "C14663" (at 63.5 107.95 90)
       (effects (font (size 1.27 1.27)) hide)
     )
@@
       (effects (font (size 1.27 1.27)) hide)
     )
+    (property "LCSC" "C14663" (at 154.94 29.21 0)
+      (effects (font (size 1.27 1.27)) hide)
+    )
     (pin "1")
     (pin "2")
@@
       (effects (font (size 1.27 1.27)) hide)
     )
+    (property "LCSC" "C407640" (at 161.29 158.75 0)
+      (effects (font (size 1.27 1.27)) hide)
+    )
     (pin "1")
     (pin "2")
@@
       (effects (font (size 1.27 1.27) italic) hide)
     )
+    (property "LCSC" "C106763" (at 120.65 184.15 0)
+      (effects (font (size 1.27 1.27)) hide)
+    )
     (pin "1")
     (pin "3")
@@
     )
     (property "Datasheet" "~" (at 39.37 132.08 0)
+      (effects (font (size 1.27 1.27)) hide)
+    )
+    (property "LCSC" "C22859" (at 39.37 132.08 90)
       (effects (font (size 1.27 1.27)) hide)
     )
@@
     (property "Datasheet" "NAU7802SGI" (at 195.58 24.13 0)
       (effects (font (size 1.27 1.27) italic) hide)
+    )
+    (property "Digikey" "NAU7802SGITR-ND " (at 201.93 29.21 0)
+      (effects (font (size 1.27 1.27)) hide)
     )
     (pin "5")
@@
       (effects (font (size 1.27 1.27)) hide)
     )
+    (property "LCSC" "C22859" (at 39.37 90.17 90)
+      (effects (font (size 1.27 1.27)) hide)
+    )
     (pin "1")
     (pin "2")
@@
       (effects (font (size 1.27 1.27)) hide)
     )
+    (property "LCSC" "C22859" (at 38.1 38.1 90)
+      (effects (font (size 1.27 1.27)) hide)
+    )
     (pin "1")
     (pin "2")
@@
     )
     (property "Datasheet" "~" (at 68.58 177.8 0)
+      (effects (font (size 1.27 1.27)) hide)
+    )
+    (property "LCSC" "C23162" (at 68.58 177.8 0)
       (effects (font (size 1.27 1.27)) hide)
     )
@@
     )
     (property "Datasheet" "https://ae-bst.resource.bosch.com/media/_tech/media/datasheets/BST-BME680-DS001.pdf" (at 43.18 179.07 0)
+      (effects (font (size 1.27 1.27)) hide)
+    )
+    (property "LCSC" "C125972" (at 43.18 173.99 0)
       (effects (font (size 1.27 1.27)) hide)
     )
@@
       (effects (font (size 1.27 1.27)) hide)
     )
+    (property "LCSC" "C407640" (at 161.29 137.16 0)
+      (effects (font (size 1.27 1.27)) hide)
+    )
     (pin "1")
     (pin "2")
@@
     )
     (property "Datasheet" "~" (at 63.5 66.04 0)
+      (effects (font (size 1.27 1.27)) hide)
+    )
+    (property "LCSC" "C14663" (at 63.5 66.04 90)
       (effects (font (size 1.27 1.27)) hide)
     )
@@
       (effects (font (size 1.27 1.27)) hide)
     )
+    (property "LCSC" "C407640" (at 161.29 180.34 0)
+      (effects (font (size 1.27 1.27)) hide)
+    )
     (pin "1")
     (pin "2")
@@
     )
     (property "Datasheet" "~" (at 38.1 121.92 0)
+      (effects (font (size 1.27 1.27)) hide)
+    )
+    (property "LCSC" "C22859" (at 38.1 121.92 90)
       (effects (font (size 1.27 1.27)) hide)
     )
@@
     (property "Datasheet" "NAU7802SGI" (at 195.58 64.77 0)
       (effects (font (size 1.27 1.27) italic) hide)
+    )
+    (property "Digikey" "NAU7802SGITR-ND " (at 201.93 69.85 0)
+      (effects (font (size 1.27 1.27)) hide)
     )
     (pin "5")
@@
       (effects (font (size 1.27 1.27)) hide)
     )
+    (property "LCSC" "C14663" (at 29.21 154.94 0)
+      (effects (font (size 1.27 1.27)) hide)
+    )
     (pin "2")
     (pin "1")
@@
       (effects (font (size 1.27 1.27)) hide)
     )
+    (property "LCSC" "C22859" (at 38.1 80.01 90)
+      (effects (font (size 1.27 1.27)) hide)
+    )
     (pin "1")
     (pin "2")
@@
       (effects (font (size 1.27 1.27)) hide)
     )
+    (property "LCSC" "C14663" (at 63.5 24.13 90)
+      (effects (font (size 1.27 1.27)) hide)
+    )
     (pin "1")
     (pin "2")
@@
     )
     (property "Datasheet" "~" (at 36.83 158.75 0)
+      (effects (font (size 1.27 1.27)) hide)
+    )
+    (property "LCSC" "C14663" (at 36.83 158.75 90)
       (effects (font (size 1.27 1.27)) hide)
     )
@@
       (effects (font (size 1.27 1.27)) hide)
     )
+    (property "LCSC" "C14663" (at 156.21 64.77 0)
+      (effects (font (size 1.27 1.27)) hide)
+    )
     (pin "1")
     (pin "2")
@@
       (effects (font (size 1.27 1.27)) hide)
     )
+    (property "LCSC" "C14663" (at 156.21 100.33 0)
+      (effects (font (size 1.27 1.27)) hide)
+    )
     (pin "1")
     (pin "2")
@@
     )
     (property "Datasheet" "~" (at 39.37 48.26 0)
+      (effects (font (size 1.27 1.27)) hide)
+    )
+    (property "LCSC" "C22859" (at 39.37 48.26 90)
       (effects (font (size 1.27 1.27)) hide)
     )
@@
       (effects (font (size 1.27 1.27) italic) hide)
     )
+    (property "LCSC" "C106763" (at 120.65 162.56 0)
+      (effects (font (size 1.27 1.27)) hide)
+    )
     (pin "1")
     (pin "3")
@@
       (effects (font (size 1.27 1.27) italic) hide)
     )
+    (property "LCSC" "C106763" (at 120.65 140.97 0)
+      (effects (font (size 1.27 1.27)) hide)
+    )
     (pin "1")
     (pin "3")
@@
       (effects (font (size 1.27 1.27)) hide)
     )
+    (property "LCSC" "C23162" (at 60.96 177.8 0)
+      (effects (font (size 1.27 1.27)) hide)
+    )

Commit message: Traces all connected v1.0
Restarted the process of routing traces (didn't account for width of 3.3V traces in first attempt). Everything is now connected for first time.
Parts:
- R18, R35, R36, R37, R38, R39, R40, R43, R44, R45, R47, R48: LCSC (none) -> C25804
- U29, U30, U31: Digikey (none) -> ED90102-ND
Changed lines of the file:
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@@
+      (effects (font (size 1.27 1.27)) hide)
+    )
+    (property "LCSC" "C25804" (at 132.08 25.4 90)
       (effects (font (size 1.27 1.27)) hide)
     )
@@
       (effects (font (size 1.27 1.27)) hide)
     )
+    (property "LCSC" "C25804" (at 110.49 43.18 90)
+      (effects (font (size 1.27 1.27)) hide)
+    )
     (pin "1")
     (pin "2")
@@
     )
     (property "Datasheet" "~" (at 63.5 113.03 0)
+      (effects (font (size 1.27 1.27)) hide)
+    )
+    (property "LCSC" "C25804" (at 63.5 113.03 90)
       (effects (font (size 1.27 1.27)) hide)
     )
@@
       (effects (font (size 1.27 1.27)) hide)
     )
+    (property "LCSC" "C25804" (at 111.76 78.74 90)
+      (effects (font (size 1.27 1.27)) hide)
+    )
     (pin "1")
     (pin "2")
@@
     )
     (property "Datasheet" "~" (at 133.35 60.96 0)
+      (effects (font (size 1.27 1.27)) hide)
+    )
+    (property "LCSC" "C25804" (at 133.35 60.96 90)
       (effects (font (size 1.27 1.27)) hide)
     )
@@
       (effects (font (size 1.27 1.27)) hide)
     )
+    (property "LCSC" "C25804" (at 158.75 25.4 90)
+      (effects (font (size 1.27 1.27)) hide)
+    )
     (pin "1")
     (pin "2")
@@
     )
     (property "Datasheet" "~" (at 63.5 29.21 0)
+      (effects (font (size 1.27 1.27)) hide)
+    )
+    (property "LCSC" "C25804" (at 63.5 29.21 90)
       (effects (font (size 1.27 1.27)) hide)
     )
@@
       (effects (font (size 1.27 1.27)) hide)
     )
+    (property "LCSC" "C25804" (at 160.02 60.96 90)
+      (effects (font (size 1.27 1.27)) hide)
+    )
     (pin "1")
     (pin "2")
@@
       (effects (font (size 1.27 1.27)) hide)
     )
+    (property "Digikey" "ED90102-ND" (at 241.3 114.3 0)
+      (effects (font (size 1.27 1.27)) hide)
+    )
     (pin "3")
     (pin "1")
@@
     )
     (property "Datasheet" "~" (at 111.76 114.3 0)
+      (effects (font (size 1.27 1.27)) hide)
+    )
+    (property "LCSC" "C25804" (at 111.76 114.3 90)
       (effects (font (size 1.27 1.27)) hide)
     )
@@
       (effects (font (size 1.27 1.27)) hide)
     )
+    (property "LCSC" "C25804" (at 63.5 71.12 90)
+      (effects (font (size 1.27 1.27)) hide)
+    )
     (pin "1")
     (pin "2")
@@
     )
     (property "Datasheet" "" (at 241.3 137.16 0)
+      (effects (font (size 1.27 1.27)) hide)
+    )
+    (property "Digikey" "ED90102-ND" (at 241.3 137.16 0)
       (effects (font (size 1.27 1.27)) hide)
     )
@@
       (effects (font (size 1.27 1.27)) hide)
     )
+    (property "Digikey" "ED90102-ND" (at 241.3 160.02 0)
+      (effects (font (size 1.27 1.27)) hide)
+    )
     (pin "3")
     (pin "1")
@@
     )
     (property "Datasheet" "~" (at 133.35 96.52 0)
+      (effects (font (size 1.27 1.27)) hide)
+    )
+    (property "LCSC" "C25804" (at 133.35 96.52 90)
       (effects (font (size 1.27 1.27)) hide)
     )
@@
       (effects (font (size 1.27 1.27)) hide)
     )
+    (property "LCSC" "C25804" (at 160.02 96.52 90)
+      (effects (font (size 1.27 1.27)) hide)
+    )
