File: Sensor-Board-KiCad7.0/Sensor-Board.kicad_sch (KiCad schematic)
At the start: 73 parts, among them J1 B4B-XH-A, U1 OPA396DCKT, U10 BME680, U13 TCA9548AMRGER, U14 OPA396DCKT, U19 MMBFJ177LT1, U2 OPA396DCKT, U20 MMBFJ177LT1, U21 OPA396DCKT, U22 OPA396DCKT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

Commit message: Fixed prelim layout errors and started traces
Fixed pad sizes for EChem sensor footprint.
Fixed silkscreen warnings.
Started routing traces in layout.
Parts:
- U23, U27, U28: footprint EChem socket:3-pin socket -> (none)
Changed lines of the file:
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@@
-    )
-  )
-  (symbol (lib_id "EChem socket:3-pin_socket") (at 198.12 137.16 0) (unit 1)
-    (in_bom yes) (on_board yes) (dnp no)
-    (property "Reference" "U27" (at 204.47 130.81 0)
-      (effects (font (size 1.27 1.27)) (justify left))
-    )
-    (property "Value" "~" (at 198.12 137.16 0)
-      (effects (font (size 1.27 1.27)))
-    )
-    (property "Footprint" "EChem socket:3-pin socket" (at 198.12 137.16 0)
-      (effects (font (size 1.27 1.27)) hide)
-    )
-    (property "Datasheet" "" (at 198.12 137.16 0)
-      (effects (font (size 1.27 1.27)) hide)
-    )
-    (pin "3")
-    (pin "2")
-    (pin "1")
-    (instances
-      (project "Sensor-Board"
-        (path "/3a986dcd-349f-492d-950a-09832b2e5abd"
-          (reference "U27") (unit 1)
-        )
-      )
     )
   )
@@
         (path "/3a986dcd-349f-492d-950a-09832b2e5abd"
           (reference "#PWR01") (unit 1)
+        )
+      )
+    )
+  )
+  (symbol (lib_id "EChem socket:3-pin_socket") (at 198.12 137.16 0) (unit 1)
+    (in_bom yes) (on_board yes) (dnp no)
+    (property "Reference" "U27" (at 204.47 130.81 0)
+      (effects (font (size 1.27 1.27)) (justify left))
+    )
+    (property "Value" "~" (at 198.12 137.16 0)
+      (effects (font (size 1.27 1.27)))
+    )
+    (property "Footprint" "" (at 198.12 137.16 0)
+      (effects (font (size 1.27 1.27)) hide)
+    )
+    (property "Datasheet" "" (at 198.12 137.16 0)
+      (effects (font (size 1.27 1.27)) hide)
+    )
+    (pin "3")
+    (pin "1")
+    (pin "2")
+    (instances
+      (project "Sensor-Board"
+        (path "/3a986dcd-349f-492d-950a-09832b2e5abd"
+          (reference "U27") (unit 1)
         )
       )
@@
     )
   )
-  (symbol (lib_id "EChem socket:3-pin_socket") (at 198.12 114.3 0) (unit 1)
-    (in_bom yes) (on_board yes) (dnp no)
-    (property "Reference" "U23" (at 204.47 107.95 0)
-      (effects (font (size 1.27 1.27)) (justify left))
-    )
-    (property "Value" "~" (at 198.12 114.3 0)
-      (effects (font (size 1.27 1.27)))
-    )
-    (property "Footprint" "EChem socket:3-pin socket" (at 198.12 114.3 0)
-      (effects (font (size 1.27 1.27)) hide)
-    )
-    (property "Datasheet" "" (at 198.12 114.3 0)
-      (effects (font (size 1.27 1.27)) hide)
-    )
-    (pin "3")
-    (pin "2")
-    (pin "1")
-    (instances
-      (project "Sensor-Board"
-        (path "/3a986dcd-349f-492d-950a-09832b2e5abd"
-          (reference "U23") (unit 1)
-        )
-      )
-    )
-  )
   (symbol (lib_id "Device:C") (at 24.13 157.48 90) (unit 1)
     (in_bom yes) (on_board yes) (dnp no)
@@
         (path "/3a986dcd-349f-492d-950a-09832b2e5abd"
           (reference "#PWR064") (unit 1)
-        )
-      )
-    )
-  )
-  (symbol (lib_id "EChem socket:3-pin_socket") (at 198.12 160.02 0) (unit 1)
-    (in_bom yes) (on_board yes) (dnp no)
-    (property "Reference" "U28" (at 204.47 153.67 0)
-      (effects (font (size 1.27 1.27)) (justify left))
-    )
-    (property "Value" "~" (at 198.12 160.02 0)
-      (effects (font (size 1.27 1.27)))
-    )
-    (property "Footprint" "EChem socket:3-pin socket" (at 198.12 160.02 0)
-      (effects (font (size 1.27 1.27)) hide)
-    )
-    (property "Datasheet" "" (at 198.12 160.02 0)
-      (effects (font (size 1.27 1.27)) hide)
-    )
-    (pin "3")
-    (pin "2")
-    (pin "1")
-    (instances
-      (project "Sensor-Board"
-        (path "/3a986dcd-349f-492d-950a-09832b2e5abd"
-          (reference "U28") (unit 1)
         )
       )
@@
     )
   )
+  (symbol (lib_id "EChem socket:3-pin_socket") (at 198.12 160.02 0) (unit 1)
+    (in_bom yes) (on_board yes) (dnp no)
+    (property "Reference" "U28" (at 204.47 153.67 0)
+      (effects (font (size 1.27 1.27)) (justify left))
+    )
+    (property "Value" "~" (at 198.12 160.02 0)
+      (effects (font (size 1.27 1.27)))
+    )
+    (property "Footprint" "" (at 198.12 160.02 0)
+      (effects (font (size 1.27 1.27)) hide)
+    )
+    (property "Datasheet" "" (at 198.12 160.02 0)
+      (effects (font (size 1.27 1.27)) hide)
+    )
+    (pin "3")
+    (pin "1")
+    (pin "2")
+    (instances
+      (project "Sensor-Board"
+        (path "/3a986dcd-349f-492d-950a-09832b2e5abd"
+          (reference "U28") (unit 1)
+        )
+      )
+    )
+  )
   (symbol (lib_id "Device:R") (at 109.22 77.47 270) (unit 1)
     (in_bom yes) (on_board yes) (dnp no)
@@
         )
       )
+    )
+  )
+  (symbol (lib_id "EChem socket:3-pin_socket") (at 198.12 114.3 0) (unit 1)
+    (in_bom yes) (on_board yes) (dnp no)
+    (property "Reference" "U23" (at 204.47 107.95 0)
+      (effects (font (size 1.27 1.27)) (justify left))
+    )
+    (property "Value" "~" (at 198.12 114.3 0)
+      (effects (font (size 1.27 1.27)))
+    )
+    (property "Footprint" "" (at 198.12 114.3 0)
+      (effects (font (size 1.27 1.27)) hide)
+    )
+    (property "Datasheet" "" (at 198.12 114.3 0)
+      (effects (font (size 1.27 1.27)) hide)
+    )
+    (pin "3")
+    (pin "1")
+    (pin "2")
+    (instances
+      (project "Sensor-Board"
+        (path "/3a986dcd-349f-492d-950a-09832b2e5abd"
+          (reference "U23") (unit 1)
+        )
+      )

Commit message: Moved components around
Moved resistors and test points around. Continued trying to route vias along the board.
Parts:
- U23, U27, U28: footprint (none) -> EChem socket:3-pin socket
Changed lines of the file:
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@@
+    )
+  )
+  (symbol (lib_id "EChem socket:3-pin_socket") (at 198.12 160.02 0) (unit 1)
+    (in_bom yes) (on_board yes) (dnp no)
+    (property "Reference" "U28" (at 204.47 153.67 0)
+      (effects (font (size 1.27 1.27)) (justify left))
+    )
+    (property "Value" "~" (at 198.12 160.02 0)
+      (effects (font (size 1.27 1.27)))
+    )
+    (property "Footprint" "EChem socket:3-pin socket" (at 198.12 160.02 0)
+      (effects (font (size 1.27 1.27)) hide)
+    )
+    (property "Datasheet" "" (at 198.12 160.02 0)
+      (effects (font (size 1.27 1.27)) hide)
+    )
+    (pin "3")
+    (pin "1")
+    (pin "2")
+    (instances
+      (project "Sensor-Board"
+        (path "/3a986dcd-349f-492d-950a-09832b2e5abd"
+          (reference "U28") (unit 1)
+        )
+      )
     )
   )
@@
         (path "/3a986dcd-349f-492d-950a-09832b2e5abd"
           (reference "#PWR020") (unit 1)
+        )
+      )
+    )
+  )
+  (symbol (lib_id "EChem socket:3-pin_socket") (at 198.12 137.16 0) (unit 1)
+    (in_bom yes) (on_board yes) (dnp no)
+    (property "Reference" "U27" (at 204.47 130.81 0)
+      (effects (font (size 1.27 1.27)) (justify left))
+    )
+    (property "Value" "~" (at 198.12 137.16 0)
+      (effects (font (size 1.27 1.27)))
+    )
+    (property "Footprint" "EChem socket:3-pin socket" (at 198.12 137.16 0)
+      (effects (font (size 1.27 1.27)) hide)
+    )
+    (property "Datasheet" "" (at 198.12 137.16 0)
+      (effects (font (size 1.27 1.27)) hide)
+    )
+    (pin "3")
+    (pin "1")
+    (pin "2")
+    (instances
+      (project "Sensor-Board"
+        (path "/3a986dcd-349f-492d-950a-09832b2e5abd"
+          (reference "U27") (unit 1)
         )
       )
@@
     )
   )
-  (symbol (lib_id "EChem socket:3-pin_socket") (at 198.12 137.16 0) (unit 1)
-    (in_bom yes) (on_board yes) (dnp no)
-    (property "Reference" "U27" (at 204.47 130.81 0)
-      (effects (font (size 1.27 1.27)) (justify left))
-    )
-    (property "Value" "~" (at 198.12 137.16 0)
-      (effects (font (size 1.27 1.27)))
-    )
-    (property "Footprint" "" (at 198.12 137.16 0)
-      (effects (font (size 1.27 1.27)) hide)
-    )
-    (property "Datasheet" "" (at 198.12 137.16 0)
-      (effects (font (size 1.27 1.27)) hide)
-    )
-    (pin "3")
-    (pin "1")
-    (pin "2")
-    (instances
-      (project "Sensor-Board"
-        (path "/3a986dcd-349f-492d-950a-09832b2e5abd"
-          (reference "U27") (unit 1)
-        )
-      )
-    )
-  )
   (symbol (lib_id "OPA396DCKT:OPA396DCKT") (at 113.03 77.47 0) (mirror x) (unit 1)
     (in_bom yes) (on_board yes) (dnp no)
@@
     )
   )
+  (symbol (lib_id "EChem socket:3-pin_socket") (at 198.12 114.3 0) (unit 1)
+    (in_bom yes) (on_board yes) (dnp no)
+    (property "Reference" "U23" (at 204.47 107.95 0)
+      (effects (font (size 1.27 1.27)) (justify left))
+    )
+    (property "Value" "~" (at 198.12 114.3 0)
+      (effects (font (size 1.27 1.27)))
+    )
+    (property "Footprint" "EChem socket:3-pin socket" (at 198.12 114.3 0)
+      (effects (font (size 1.27 1.27)) hide)
+    )
+    (property "Datasheet" "" (at 198.12 114.3 0)
+      (effects (font (size 1.27 1.27)) hide)
+    )
+    (pin "3")
+    (pin "1")
+    (pin "2")
+    (instances
+      (project "Sensor-Board"
+        (path "/3a986dcd-349f-492d-950a-09832b2e5abd"
+          (reference "U23") (unit 1)
+        )
+      )
+    )
+  )
   (symbol (lib_id "Device:R") (at 161.29 180.34 0) (mirror x) (unit 1)
     (in_bom yes) (on_board yes) (dnp no)
@@
     )
   )
-  (symbol (lib_id "EChem socket:3-pin_socket") (at 198.12 160.02 0) (unit 1)
-    (in_bom yes) (on_board yes) (dnp no)
-    (property "Reference" "U28" (at 204.47 153.67 0)
-      (effects (font (size 1.27 1.27)) (justify left))
-    )
-    (property "Value" "~" (at 198.12 160.02 0)
-      (effects (font (size 1.27 1.27)))
-    )
-    (property "Footprint" "" (at 198.12 160.02 0)
-      (effects (font (size 1.27 1.27)) hide)
-    )
-    (property "Datasheet" "" (at 198.12 160.02 0)
-      (effects (font (size 1.27 1.27)) hide)
-    )
-    (pin "3")
-    (pin "1")
-    (pin "2")
-    (instances
-      (project "Sensor-Board"
-        (path "/3a986dcd-349f-492d-950a-09832b2e5abd"
-          (reference "U28") (unit 1)
-        )
-      )
-    )
-  )
   (symbol (lib_id "Device:R") (at 109.22 77.47 270) (unit 1)
     (in_bom yes) (on_board yes) (dnp no)
@@
         )
       )
-    )
-  )
-  (symbol (lib_id "EChem socket:3-pin_socket") (at 198.12 114.3 0) (unit 1)
-    (in_bom yes) (on_board yes) (dnp no)
-    (property "Reference" "U23" (at 204.47 107.95 0)
-      (effects (font (size 1.27 1.27)) (justify left))
-    )
-    (property "Value" "~" (at 198.12 114.3 0)
-      (effects (font (size 1.27 1.27)))
-    )
-    (property "Footprint" "" (at 198.12 114.3 0)
-      (effects (font (size 1.27 1.27)) hide)
-    )
-    (property "Datasheet" "" (at 198.12 114.3 0)
-      (effects (font (size 1.27 1.27)) hide)
-    )
-    (pin "3")
-    (pin "1")
-    (pin "2")
-    (instances
-      (project "Sensor-Board"
-        (path "/3a986dcd-349f-492d-950a-09832b2e5abd"
-          (reference "U23") (unit 1)
-        )
-      )

Commit message: Added some part #
Added part numbers for resistors, capacitors, MOSFETS
Parts:
- C1, C19, C2, C20, C21, C3, C8, C9: LCSC (none) -> C14663
- R1, R2, R3, R4, R5, R54, R55, R56, R57, R6, R69, R9: LCSC (none) -> C25804
- R19, R20, R21, R22, R23, R24, R25, R26, R27, R28, R29, R30, R31, R32, R33, R34: LCSC (none) -> C23162
- R41, R42, R46: LCSC (none) -> C407640
- R52, R53, R67, R68, R7, R8: LCSC (none) -> C22859
- U10: LCSC (none) -> C125972
- U25, U4: Digikey (none) -> NAU7802SGITR-ND
Changed lines of the file:
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@@
+      (effects (font (size 1.27 1.27)) hide)
+    )
+    (property "LCSC" "C25804" (at 60.96 69.85 90)
       (effects (font (size 1.27 1.27)) hide)
     )
@@
     (property "Datasheet" "NAU7802SGI" (at 195.58 22.86 0)
       (effects (font (size 1.27 1.27) italic) hide)
+    )
+    (property "Digikey" "NAU7802SGITR-ND " (at 201.93 27.94 0)
+      (effects (font (size 1.27 1.27)) hide)
     )
     (pin "5")
@@
     )
     (property "Datasheet" "~" (at 157.48 95.25 0)
+      (effects (font (size 1.27 1.27)) hide)
+    )
+    (property "LCSC" "C25804" (at 157.48 95.25 90)
       (effects (font (size 1.27 1.27)) hide)
     )
@@
       (effects (font (size 1.27 1.27)) hide)
     )
+    (property "LCSC" "C23162" (at 254 135.89 90)
+      (effects (font (size 1.27 1.27)) hide)
+    )
     (pin "1")
     (pin "2")
@@
       (effects (font (size 1.27 1.27)) hide)
     )
+    (property "LCSC" "C22859" (at 36.83 46.99 90)
+      (effects (font (size 1.27 1.27)) hide)
+    )
     (pin "1")
     (pin "2")
@@
     )
     (property "Datasheet" "https://ae-bst.resource.bosch.com/media/_tech/media/datasheets/BST-BME680-DS001.pdf" (at 30.48 177.8 0)
+      (effects (font (size 1.27 1.27)) hide)
+    )
+    (property "LCSC" "C125972" (at 30.48 172.72 0)
       (effects (font (size 1.27 1.27)) hide)
     )
@@
       (effects (font (size 1.27 1.27)) hide)
     )
+    (property "LCSC" "C23162" (at 254 118.11 90)
+      (effects (font (size 1.27 1.27)) hide)
+    )
     (pin "1")
     (pin "2")
@@
     )
     (property "Datasheet" "~" (at 130.81 59.69 0)
+      (effects (font (size 1.27 1.27)) hide)
+    )
+    (property "LCSC" "C25804" (at 130.81 59.69 90)
       (effects (font (size 1.27 1.27)) hide)
     )
@@
       (effects (font (size 1.27 1.27)) hide)
     )
+    (property "LCSC" "C407640" (at 161.29 137.16 0)
+      (effects (font (size 1.27 1.27)) hide)
+    )
     (pin "1")
     (pin "2")
@@
     )
     (property "Datasheet" "~" (at 60.96 64.77 0)
+      (effects (font (size 1.27 1.27)) hide)
+    )
+    (property "LCSC" "C14663" (at 60.96 64.77 90)
       (effects (font (size 1.27 1.27)) hide)
     )
@@
       (effects (font (size 1.27 1.27)) hide)
     )
+    (property "LCSC" "C25804" (at 109.22 113.03 90)
+      (effects (font (size 1.27 1.27)) hide)
+    )
     (pin "1")
     (pin "2")
@@
       (effects (font (size 1.27 1.27)) hide)
     )
+    (property "LCSC" "C23162" (at 226.06 110.49 90)
+      (effects (font (size 1.27 1.27)) hide)
+    )
     (pin "1")
     (pin "2")
@@
       (effects (font (size 1.27 1.27)) hide)
     )
+    (property "LCSC" "C14663" (at 152.4 27.94 0)
+      (effects (font (size 1.27 1.27)) hide)
+    )
     (pin "1")
     (pin "2")
@@
     )
     (property "Datasheet" "~" (at 35.56 120.65 0)
+      (effects (font (size 1.27 1.27)) hide)
+    )
+    (property "LCSC" "C22859" (at 35.56 120.65 90)
       (effects (font (size 1.27 1.27)) hide)
     )
@@
       (effects (font (size 1.27 1.27)) hide)
     )
+    (property "LCSC" "C407640" (at 161.29 158.75 0)
+      (effects (font (size 1.27 1.27)) hide)
+    )
     (pin "1")
     (pin "2")
@@
       (effects (font (size 1.27 1.27)) hide)
     )
+    (property "LCSC" "C23162" (at 48.26 176.53 0)
+      (effects (font (size 1.27 1.27)) hide)
+    )
     (pin "1")
     (pin "2")
@@
       (effects (font (size 1.27 1.27)) hide)
     )
+    (property "LCSC" "C23162" (at 254 130.81 90)
+      (effects (font (size 1.27 1.27)) hide)
+    )
     (pin "1")
     (pin "2")
@@
       (effects (font (size 1.27 1.27)) hide)
     )
+    (property "LCSC" "C14663" (at 24.13 157.48 90)
+      (effects (font (size 1.27 1.27)) hide)
+    )
     (pin "1")
     (pin "2")
@@
       (effects (font (size 1.27 1.27)) hide)
     )
+    (property "LCSC" "C22859" (at 36.83 88.9 90)
+      (effects (font (size 1.27 1.27)) hide)
+    )
     (pin "1")
     (pin "2")
@@
     )
     (property "Datasheet" "~" (at 36.83 130.81 0)
+      (effects (font (size 1.27 1.27)) hide)
+    )
+    (property "LCSC" "C22859" (at 36.83 130.81 90)
       (effects (font (size 1.27 1.27)) hide)
     )
@@
       (effects (font (size 1.27 1.27)) hide)
     )
+    (property "LCSC" "C407640" (at 161.29 180.34 0)
+      (effects (font (size 1.27 1.27)) hide)
+    )
     (pin "1")
     (pin "2")
@@
       (effects (font (size 1.27 1.27)) hide)
     )
+    (property "LCSC" "C23162" (at 254 115.57 90)
+      (effects (font (size 1.27 1.27)) hide)
+    )
     (pin "1")
     (pin "2")
@@
     )
     (property "Datasheet" "~" (at 254 110.49 0)
+      (effects (font (size 1.27 1.27)) hide)
+    )
+    (property "LCSC" "C23162" (at 254 110.49 90)
       (effects (font (size 1.27 1.27)) hide)
     )
@@
       (effects (font (size 1.27 1.27)) hide)
     )
+    (property "LCSC" "C23162" (at 55.88 176.53 0)
+      (effects (font (size 1.27 1.27)) hide)
+    )
     (pin "2")
     (pin "1")
@@
       (effects (font (size 1.27 1.27)) hide)
     )
+    (property "LCSC" "C25804" (at 156.21 24.13 90)
+      (effects (font (size 1.27 1.27)) hide)
+    )
     (pin "1")
     (pin "2")
@@
       (effects (font (size 1.27 1.27)) hide)
     )
+    (property "LCSC" "C14663" (at 16.51 153.67 0)
+      (effects (font (size 1.27 1.27)) hide)
+    )
     (pin "2")
     (pin "1")
@@
       (effects (font (size 1.27 1.27)) hide)
     )
+    (property "LCSC" "C25804" (at 109.22 77.47 90)
+      (effects (font (size 1.27 1.27)) hide)
+    )
     (pin "1")
     (pin "2")
@@
     )
     (property "Datasheet" "~" (at 35.56 78.74 0)
+      (effects (font (size 1.27 1.27)) hide)
+    )
+    (property "LCSC" "C22859" (at 35.56 78.74 90)
       (effects (font (size 1.27 1.27)) hide)
     )
@@
       (effects (font (size 1.27 1.27)) hide)
     )
+    (property "LCSC" "C14663" (at 60.96 106.68 90)
+      (effects (font (size 1.27 1.27)) hide)
+    )
     (pin "1")
     (pin "2")
@@
       (effects (font (size 1.27 1.27)) hide)
     )
+    (property "LCSC" "C25804" (at 130.81 95.25 90)
+      (effects (font (size 1.27 1.27)) hide)
+    )
     (pin "1")
     (pin "2")
@@
       (effects (font (size 1.27 1.27)) hide)
     )
+    (property "LCSC" "C23162" (at 254 138.43 90)
+      (effects (font (size 1.27 1.27)) hide)
+    )
     (pin "1")
     (pin "2")
@@
       (effects (font (size 1.27 1.27)) hide)
     )
+    (property "LCSC" "C25804" (at 157.48 59.69 90)
+      (effects (font (size 1.27 1.27)) hide)
+    )
     (pin "1")
     (pin "2")
@@
       (effects (font (size 1.27 1.27)) hide)
     )
+    (property "LCSC" "C23162" (at 254 123.19 90)
+      (effects (font (size 1.27 1.27)) hide)
+    )
     (pin "1")
     (pin "2")
@@
       (effects (font (size 1.27 1.27)) hide)
     )
+    (property "LCSC" "C25804" (at 129.54 24.13 90)
+      (effects (font (size 1.27 1.27)) hide)
+    )
     (pin "1")
     (pin "2")
@@
       (effects (font (size 1.27 1.27)) hide)
     )
+    (property "LCSC" "C23162" (at 254 128.27 90)
+      (effects (font (size 1.27 1.27)) hide)
+    )
     (pin "1")
     (pin "2")
@@
       (effects (font (size 1.27 1.27)) hide)
     )
+    (property "LCSC" "C23162" (at 254 120.65 90)
+      (effects (font (size 1.27 1.27)) hide)
+    )
     (pin "1")
     (pin "2")
@@
       (effects (font (size 1.27 1.27)) hide)
     )
+    (property "LCSC" "C22859" (at 35.56 36.83 90)
+      (effects (font (size 1.27 1.27)) hide)
+    )
     (pin "1")
     (pin "2")
@@
     )
     (property "Datasheet" "~" (at 60.96 22.86 0)
+      (effects (font (size 1.27 1.27)) hide)
+    )
+    (property "LCSC" "C14663" (at 60.96 22.86 90)
       (effects (font (size 1.27 1.27)) hide)
     )
@@
       (effects (font (size 1.27 1.27)) hide)
     )
+    (property "LCSC" "C14663" (at 153.67 63.5 0)
+      (effects (font (size 1.27 1.27)) hide)
+    )
     (pin "1")
     (pin "2")
@@
       (effects (font (size 1.27 1.27)) hide)
     )
+    (property "LCSC" "C25804" (at 60.96 27.94 90)
+      (effects (font (size 1.27 1.27)) hide)
+    )
     (pin "1")
     (pin "2")
@@
       (effects (font (size 1.27 1.27)) hide)
     )
+    (property "LCSC" "C25804" (at 107.95 41.91 90)
+      (effects (font (size 1.27 1.27)) hide)
+    )
     (pin "1")
     (pin "2")
@@
     )
     (property "Datasheet" "~" (at 254 133.35 0)
+      (effects (font (size 1.27 1.27)) hide)
+    )
+    (property "LCSC" "C23162" (at 254 133.35 90)
       (effects (font (size 1.27 1.27)) hide)
     )
@@
       (effects (font (size 1.27 1.27)) hide)
     )
+    (property "LCSC" "C23162" (at 254 125.73 90)
+      (effects (font (size 1.27 1.27)) hide)
+    )
     (pin "1")
     (pin "2")
@@
     )
     (property "Datasheet" "~" (at 226.06 113.03 0)
+      (effects (font (size 1.27 1.27)) hide)
+    )
+    (property "LCSC" "C23162" (at 226.06 113.03 90)
       (effects (font (size 1.27 1.27)) hide)
     )
@@
     (property "Datasheet" "NAU7802SGI" (at 195.58 63.5 0)
       (effects (font (size 1.27 1.27) italic) hide)
+    )
+    (property "Digikey" "NAU7802SGITR-ND " (at 201.93 68.58 0)
+      (effects (font (size 1.27 1.27)) hide)
     )
     (pin "5")
@@
       (effects (font (size 1.27 1.27)) hide)
     )
+    (property "LCSC" "C25804" (at 60.96 111.76 90)
+      (effects (font (size 1.27 1.27)) hide)
+    )
     (pin "1")
     (pin "2")
@@
       (effects (font (size 1.27 1.27)) hide)
     )
+    (property "LCSC" "C14663" (at 153.67 99.06 0)
+      (effects (font (size 1.27 1.27)) hide)
+    )
     (pin "1")
     (pin "2")
@@
       (effects (font (size 1.27 1.27)) hide)
     )
+    (property "LCSC" "C23162" (at 254 113.03 90)
+      (effects (font (size 1.27 1.27)) hide)
+    )
