File: Motherboard KiCad7.0/Motherboard/Motherboard.kicad_sch (KiCad schematic)
At the start: 59 parts, among them J1 USB_B_Micro, J2 SWD_01x04_Pin, Q7 AO4447A, SW1 SW_STM_RESET, SW2 SW_STM_BOOT_MODE, U1 STM32F103CBT6, U2 AMS1117-3.3, U3 LM66100DCKR, U4 LM66100DCKR, U5 LM66100DCKR, U6 LMR51430XDDCR, Y1 X322516MMB4SI

Commit message: Added missing sensors
Added MPU6050, MS5607, and KX134 for altimeter. Fixed library issues. Re-added part numbers. Started fixing layout.
Parts:
- removed C18: 100nF, Capacitor_SMD:C_0603_1608Metric, symbol Device:C
- removed C22: 100uF, Capacitor_SMD:CP_Elec_6.3x5.9, symbol Device:C_Polarized
- removed D11, D3: WS2812B, LED_SMD:LED_WS2812B_PLCC4_5.0x5.0mm_P3.2mm, symbol LED:WS2812B
- removed D4: DB_LED (YLW), LED_SMD:LED_0603_1608Metric, symbol Device:LED
- removed J2: SWD_01x04_Pin, SWD_Header:SWD_PinHeader_1x04_P2.54mm_Horizontal, symbol QRET_Edge_Connector:SWD_01x04_Pin
- removed J? (x2): 430450200, CONN 0430450200:CON_430450200_MOL, symbol CONN 0430450200:430450200
- removed L1: 5.6uH, Inductor_SMD:L_Bourns_SRN8040TA, symbol Device:L
- removed Q7: AO4447A, Package_SO:SOIC-8_3.9x4.9mm_P1.27mm, symbol Transistor_FET:IRF7404
- removed R19, R3: 100k, Resistor_SMD:R_0603_1608Metric, symbol Device:R
- removed R20: 22k, Resistor_SMD:R_0603_1608Metric, symbol Device:R
- removed SW2: SW_STM_BOOT_MODE, PTS636:PTS636_SK43_SMTR_LFS, symbol Switch:SW_Push
- removed TP5: TP_VUSB, TestPoint:TestPoint_Pad_1.5x1.5mm, symbol Connector:TestPoint
- removed TP6: TP_VSWD, TestPoint:TestPoint_Pad_1.5x1.5mm, symbol Connector:TestPoint
- removed TP7: TP_MUX, TestPoint:TestPoint_Pad_1.5x1.5mm, symbol Connector:TestPoint
- removed TP8: TP_BATT1, TestPoint:TestPoint_Pad_2.0x2.0mm, symbol Connector:TestPoint
- removed TP9: TP_3.3V_A, TestPoint:TestPoint_Pad_2.0x2.0mm, symbol Connector:TestPoint
- removed U3, U4, U5: LM66100DCKR, LMR66100:SC-70-6, symbol QRET_Buck_PSU:LM66100DCKR
- removed U6: LMR51430XDDCR, Package_TO_SOT_SMD:SOT-23-6_Handsoldering, symbol QRET_Buck_PSU-symbols:LMR51430XDDCR
- removed U?: DEV-13743, DEV-13743:MODULE_DEV-13743, symbol DEV-13743:DEV-13743
- added BZ1: PKM13EPYH4000, Buzzer_12.6x9.5RM5.0:Buzzer_12.6x9.5RM5.0, symbol Device:Buzzer
- added C22, C23: 100nF, Capacitor_SMD:C_0603_1608Metric, symbol Device:C
- added C24: 2.2nF, Capacitor_SMD:C_0603_1608Metric, symbol Device:C
- added D1, D2: WS2812B, LED_SMD:LED_WS2812B_PLCC4_5.0x5.0mm_P3.2mm, symbol LED:WS2812B
- added D10, D12, D13, D14, D15, D16, D17: 1N5819WS, Diode_SMD:D_SOD-323, symbol Diode:1N5819WS
- added D3: LED, LED_SMD:LED_0603_1608Metric, symbol Device:LED
- added H1, H2: MountingHole, Rod_Mounting_Hole_6.7564mm:Rod_Mounting_Hole_6.7564mm, symbol Mechanical:MountingHole
- added J10, J11, J12, J4, J6, J7: 430450200, CON_430450200_MOL, symbol CONN 0430450200:430450200
- added J2: SWD_01x04_Pin, SWD_Header:SWD_PinHeader_1x04_P2.54mm_Horizontal, symbol EdgeConnector:SWD_01x04_Pin
- added J3: 430450200, CONN 0430450200:CON_430450200_MOL, symbol CONN 0430450200:430450200
- added J5: B04B-XASK-1, CONN_B04B-XASK-1_JST, symbol B04B_XASK_1:B04B-XASK-1
- added PS1: K7803JT-500R3-LB, K7805JT_500R3:K78_JT-500R3_MNS, symbol K7812JT-500R3-LB:K7812JT-500R3-LB
- added Q1: AO4447A, Package_TO_SOT_SMD:SOT-23, symbol Transistor_FET:AO3400A
- added Q10, Q11, Q12, Q13, Q8, Q9: AO3400A, Package_TO_SOT_SMD:SOT-23, symbol Transistor_FET:AO3400A
- added R21, R23, R24, R25, R26, R27, R5: 10k, Resistor_SMD:R_0603_1608Metric, symbol Device:R
- added R22, R28, R29, R30, R31, R32: 510R, Resistor_SMD:R_0603_1608Metric, symbol Device:R
- added R33: 1k, Resistor_SMD:R_0603_1608Metric, symbol Device:R
- added R4: 30k, Resistor_SMD:R_0603_1608Metric, symbol Device:R
- added R7: 560, Resistor_SMD:R_0603_1608Metric, symbol Device:R
- added SW3: SW_STM_BOOT_MODE, Button_Switch_SMD:SW_Push_1P1T_XKB_TS-1187A, symbol Switch:SW_MEC_5G
- added U10: KX134-1211, Package_LGA:LGA-12_2x2mm_P0.5mm, symbol KX134-1211:KX134-1211
- added U3, U4, U5: LM66100DCKR, LMR66100:SC-70-6_Handsoldering, symbol QRET_Buck_PSU-symbols:LM66100DCKR
- added U7: Micro_SD_Reader, MicroSD Card Reader:MicroSD Card Reader, symbol MicroSD Card Reader:Micro_SD_Reader
- added U8: MPU-6050, Sensor_Motion:InvenSense_QFN-24_4x4mm_P0.5mm, symbol Sensor_Motion:MPU-6050
- added U9: MS560702BA03-50, MS5607_Handsolder:MS5607_Handsolder, symbol Sensor_Pressure:MS5607-02BA
- C10, C11: footprint Capacitor_SMD:CP_Elec_4x5.4 -> Capacitor_SMD:C_0805_2012Metric
- C17: value 4.7uF -> 100nF; footprint Capacitor_SMD:C_0805_2012Metric -> Capacitor_SMD:C_0603_1608Metric; LCSC C1779 -> C14663
- C20: value 22uF -> 100nF; footprint Capacitor_SMD:C_0805_2012Metric -> Capacitor_SMD:C_0603_1608Metric; LCSC C45783 -> C14663
- C21: value 22uF -> 10nF; footprint Capacitor_SMD:C_0805_2012Metric -> Capacitor_SMD:C_0603_1608Metric; LCSC C45783 -> C57112
- J1: footprint footprints:USB_Micro-B_Amphenol_10118194_Horizontal -> USB_Micro-B_Amphenol_10118194_Horizontal:USB_Micro-B_Amphenol_10118194_Horizontal
- R6: value 560R -> 100k; LCSC C23204 -> C25803
- SW1: footprint PTS636:PTS636_SK43_SMTR_LFS -> Button_Switch_SMD:SW_Push_1P1T_XKB_TS-1187A
- TP1: value TP_PB5 -> TP_VBUCK
- TP2: value TP_PB6 -> TP_VREGUSB
- TP3: value TP_PB7 -> TP_VSWD
- TP4: value TP_VSTACK -> TestPoint; footprint TestPoint:TestPoint_Pad_1.5x1.5mm -> TestPoint:TestPoint_Pad_1.0x1.0mm
Connections:
- net BATT_A is gone; now on net +3.3V: C17.1
- net +3.3V: now also C19.2, C20.1, C21.2, C22.1, D1.1 (VDD), D12.2 (A), D2.1 (VDD), J5.4, SW3.3 (B), SW3.4 (B), U10.1 (SDO/ADDR), U10.10 (nCS), U10.3 (IO_VDD), U10.7 (VDD), U3.3 (*CE), U3.6 (VOUT), U4.3 (*CE), U4.6 (VOUT), U5.3 (*CE), U5.6 (VOUT), U7.2 (3.3V), U8.13 (VDD), U8.8 (VLOGIC), U8.9 (AD0), U9.1 (VDD), U9.2 (PS), U9.4 (CSB), U9.5 (CSB)
- net BATT_SENSE: now also TP4.1, R4.2, R5.1
- net BOOT0: now also R6.1, SW3.1 (A), SW3.2 (A); no longer R1.2
- net BOOT1: now also R1.2
- net BUZZER: now also R21.2, R22.2
- net DB_LED: now also R7.2; no longer R6.2
- net GND: now also C19.1, C21.1, R6.2, C22.2, C23.2, C24.2, D1.3 (VSS), D2.3 (VSS), D3.1 (K), J2.1 (GND), J5.1, J7.1, PS1.4 (GND), Q1.1 (G), Q10.2 (S), Q11.2 (S), Q12.2 (S), Q13.2 (S), Q8.2 (S), Q9.2 (S), R21.1, R23.1, R24.1, R25.1, R26.1, R27.1, R5.2, U10.4 (TRIG), U10.8 (GND), U10.9 (GND), U3.2 (GND), U3.5 (ST), U4.2 (GND), U4.5 (ST), U5.2 (GND), U5.5 (ST), U7.1 (GND), U8.1 (CLKIN), U8.11 (FSYNC), U8.18 (GND), U9.3 (GND); no longer C21.2
- net Pump: now also U1.29 (PA8), R27.2, R32.2; no longer U1.14 (PA4)
- net RGB_DATA: now also D1.4 (DIN)
- net SWCLK: now also J2.4 (SWCLK)
- net SWDIO: now also J2.3 (SWDIO)
- net Sol_0: now also R23.2, R28.2
- net Sol_1: now also R24.2, R29.2
- net Sol_2: now also R25.2, R30.2
- net Sol_3: now also R26.2, R31.2
- net V_REGUSB: now also TP2.1, U4.1 (VIN)
- net V_SWD: now also TP3.1, J2.2 (3V3), U5.1 (VIN)
- net GYRO_INT: now reaches U1.43 (PB7)
- net GYRO_INT: now also U8.12 (INT); no longer TP3.1
- net ACCEL_INT1: now reaches U1.41 (PB5)
- net ACCEL_INT1: now also U10.5 (INT1); no longer TP1.1
- net ACCEL_INT2: now reaches U1.42 (PB6)
- net ACCEL_INT2: now also U10.6 (INT2); no longer TP2.1
- net SD_CLK: now reaches U1.15 (PA5)
- net SD_CLK: now also U7.5 (CLK)
- net SD_MISO: now reaches U1.16 (PA6)
- net SD_MISO: now also U7.3 (MISO)
- net SD_MOSI: now reaches U1.17 (PA7)
- net SD_MOSI: now also U7.4 (MOSI)
- net SDA: now reaches U1.21 (PB10)
- net SDA: now also J5.2, U10.2 (SDI/SDA), U8.24 (SDA), U9.7 (SDI/SDA)
- net SCL: now reaches U1.22 (PB11)
- net SCL: now also J5.3, U10.12 (SCLK/SCL), U8.23 (SCL), U9.8 (SCLK)
- removed net 3.3V_A: C20.1, C21.1
- net CS_FL: no longer names the net of U1.25 (PB12)
- net CURR_SENSE: no longer names the net of U1.19 (PB1)
- net SCK_FL: no longer names the net of U1.26 (PB13)
- net V_PSU renamed V_BUCK
- net V_BUCK: now also TP1.1, PS1.3 (+VO), U3.1 (VIN); no longer TP4.1
- new net: Q12.1 (G), R31.1
- new net: C23.1, U8.10 (REGOUT)
- new net: C24.1, U8.20 (CPOUT)
- new net: D15.2 (A), J10.2, Q11.3 (D)
- new net: J6.2, Q1.2 (S)
- new net: Q8.1 (G), R22.1
- new net: BZ1.2 (-), Q8.3 (D), R33.1
- new net: D3.2 (A), R7.1
- new net: J6.1, J7.2
- new net: D17.2 (A), J12.2, Q13.3 (D)
- new net: Q11.1 (G), R30.1
- new net: D16.2 (A), J11.2, Q12.3 (D)
- new net: Q13.1 (G), R32.1
- new net: BZ1.1 (+), D10.1 (K), D12.1 (K), R33.2
- new net: Q9.1 (G), R28.1
- new net: D13.2 (A), J3.2, Q9.3 (D)
- new net: D1.2 (DOUT), D2.4 (DIN)
- new net: Q10.1 (G), R29.1
- new net: D14.2 (A), J4.2, Q10.3 (D)
- new net +BATT: D10.2 (A), D13.1 (K), D14.1 (K), D15.1 (K), D16.1 (K), D17.1 (K), J10.1, J11.1, J12.1, J3.1, J4.1, PS1.1 (+VIN), Q1.3 (D), R4.1
- new net SD_CS: U1.14 (PA4), U7.6 (CS)
Other:
- removed sheet Motherboard P2
- note added: "100nF cap should be as close to VDD as possible"
- note added: "Air Pump"
- note added: "Battery monitoring"
- note added: "Buzzer"
- note added: "I2C ADDRESS: 0x1E (ADDR 0.0V) >0x1F (ADDR 3.3V)"
- note added: "I2C ADDRESS: 0x77 (CSB 0.0V) >0x76 (CSB 3.3V)"
- note added: "I2C Connector"
- note added: "KX134 Accelerometer (I2C)"
- note added: "MAKE SURE AROUND EDGE OF PCB"
- note added: "MPU6050 Gyroscope (I2C)"
- note added: "MS5607 Pressure Sensor (I2C)"
- note added: "Mounting holes"
- note added: "Place in center of PCB"
- note added: "SD Card Reader (SPI)"
- note added: "Solenoid Valves"
- note removed: "FOLLOW LAYOUT EXAMPLE (9.4.2) FROM DATASHEET LMR51430: PFM @ 500kHz (simpler routing & higher efficiency)"
- note removed: "Max Output: 2.5A"
- note removed: "Rfbt=100k, Rfbb=22k Vout = ((Rfbt*0.6)/Rfbb)+0.6 Vout = 3.327V"
- company: (none) -> Queen's Rocket Engineering Team
- title: (none) -> Motherboard
- moved on the sheet: C1, C10, C11, C12, C13, C2, C3, C4, C5, C6, C7, C8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

Commit message: Finished layout and added some part numbers
Parts:
- PS1: Digikey (none) -> 2725-K7803JT-500R3-LBCT-ND
- U10: LCSC (none) -> C2157908
Changed lines of the file:
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@@
       (effects (font (size 1.27 1.27) italic) hide)
+    )
+    (property "LCSC" "C2157908" (at 86.36 86.36 0)
+      (effects (font (size 1.27 1.27)) hide)
     )
     (pin "12")
@@
       (effects (font (size 1.27 1.27)) (justify bottom) hide)
     )
-    (pin "1")
+    (property "Digikey" "2725-K7803JT-500R3-LBCT-ND" (at 179.07 100.33 0)
+      (effects (font (size 1.27 1.27)) hide)
+    )
+    (pin "1")
